File: cranklight/cranklight.sch (KiCad schematic (older format))
At the start: 23 parts, among them J1 Battery, J2 Bulb socket, Q1 Q_NMOS_GDS, SW1 SW_4PDT, U1 WeMos_mini, U2 PTN04050CAD

Commit message: Add fixes: move PTC, add charging connector, use switch as a simple switch
Parts:
- removed unit 3 of SW1
- removed unit 4 of SW1
- added J3: Charge, Pin_Headers:Pin_Header_Angled_1x02_Pitch2.54mm, symbol Connector_Generic:Conn_01x02
- R4: value 1M -> 100k
Connections:
- wire segments 44 -> 33
Changed lines of the file:
@@
 Sheet 1 1
 Title "Chernobyl cranklight"
-Date "2018-06-05"
+Date "2018-06-18"
 Rev "1"
 Comp "Albertas Mickėnas"
@@
 $EndComp
 $Comp
-L power:+BATT #PWR0104
-U 1 1 5B168006
-P 8500 5200
-F 0 "#PWR0104" H 8500 5050 50  0001 C CNN
-F 1 "+BATT" H 8350 5250 50  0000 C CNN
-F 2 "" H 8500 5200 50  0001 C CNN
-F 3 "" H 8500 5200 50  0001 C CNN
-	1    8500 5200
-	1    0    0    -1
-$EndComp
-$Comp
 L Device:R R3
 U 1 1 5B168086
@@
 P 8500 7100
 F 0 "R4" H 8431 7054 50  0000 R CNN
-F 1 "1M" H 8431 7145 50  0000 R CNN
+F 1 "100k" H 8431 7145 50  0000 R CNN
 F 2 "Resistors_SMD:R_0805_2012Metric_Pad1.33x1.40mm_HandSolder" V 8430 7100 50  0001 C CNN
 F 3 "~" H 8500 7100 50  0001 C CNN
@@
 	9100 7250 9100 7150
 Connection ~ 9100 7250
-Wire Wire Line
-	9100 6350 9100 5850
-Wire Wire Line
-	9900 6350 10150 6350
-Wire Wire Line
-	10150 6350 10150 6750
-Wire Wire Line
-	9900 6250 10250 6250
-Wire Wire Line
-	10250 6250 10250 7250
-Wire Wire Line
-	10250 7250 9100 7250
 $Comp
 L power:GND #PWR0106
@@
 L Device:Polyfuse F1
 U 1 1 5B169393
-P 9800 6750
-F 0 "F1" V 9575 6750 50  0000 C CNN
-F 1 "Polyfuse" V 9666 6750 50  0000 C CNN
-F 2 "Fuse_Holders_and_Fuses:Fuse_Littelfuse-LVR100" H 9850 6550 50  0001 L CNN
-F 3 "~" H 9800 6750 50  0001 C CNN
-F 4 "LVR100S" H 9800 6750 50  0001 C CNN "PartNo"
-F 5 "Littlefuse" H 9800 6750 50  0001 C CNN "Manufacturer"
-F 6 "Mouser/650-LVR100S" H 9800 6750 50  0001 C CNN "Distributor"
-	1    9800 6750
-	0    1    1    0
-$EndComp
-Wire Wire Line
-	9950 6750 10150 6750
-Wire Wire Line
-	9100 6750 9650 6750
+P 9100 5500
+F 0 "F1" V 8875 5500 50  0000 C CNN
+F 1 "Polyfuse" V 8966 5500 50  0000 C CNN
+F 2 "Fuse_Holders_and_Fuses:Fuse_Littelfuse-LVR100" H 9150 5300 50  0001 L CNN
+F 3 "~" H 9100 5500 50  0001 C CNN
+F 4 "LVR100S" H 9100 5500 50  0001 C CNN "PartNo"
+F 5 "Littlefuse" H 9100 5500 50  0001 C CNN "Manufacturer"
+F 6 "Mouser/650-LVR100S" H 9100 5500 50  0001 C CNN "Distributor"
+	1    9100 5500
+	-1   0    0    1
+$EndComp
 $Comp
 L Device:C C4
@@
 	4500 6550 5250 6550
 NoConn ~ 4950 6250
-Wire Wire Line
-	9100 5350 9100 5750
-Connection ~ 9100 5750
-Wire Wire Line
-	9900 6450 9900 6350
 $Comp
 L power:+5V #PWR02
 U 1 1 5B19B8F9
-P 8500 5450
-F 0 "#PWR02" H 8500 5300 50  0001 C CNN
-F 1 "+5V" H 8350 5500 50  0000 C CNN
-F 2 "" H 8500 5450 50  0001 C CNN
-F 3 "" H 8500 5450 50  0001 C CNN
-	1    8500 5450
-	1    0    0    -1
-$EndComp
-$Comp
-L dp3t:SW_4PDT SW1
-U 3 1 5B19C6FA
-P 8900 5350
-F 0 "SW1" H 8900 5635 50  0000 C CNN
-F 1 "SW_4PDT" H 8900 5544 50  0000 C CNN
-F 2 "wemos:4PDT" H 8900 5350 50  0001 C CNN
-F 3 "" H 8900 5350 50  0001 C CNN
-	3    8900 5350
-	-1   0    0    -1
-$EndComp
-$Comp
-L dp3t:SW_4PDT SW1
-U 4 1 5B19CC8F
-P 9700 6350
-F 0 "SW1" H 9700 6635 50  0000 C CNN
-F 1 "SW_4PDT" H 9700 6544 50  0000 C CNN
-F 2 "wemos:4PDT" H 9700 6350 50  0001 C CNN
-F 3 "" H 9700 6350 50  0001 C CNN
-	4    9700 6350
-	1    0    0    -1
-$EndComp
-Wire Wire Line
-	9100 6350 9500 6350
-Wire Wire Line
-	8500 5450 8700 5450
+P 9100 5350
+F 0 "#PWR02" H 9100 5200 50  0001 C CNN
+F 1 "+5V" H 8950 5400 50  0000 C CNN
+F 2 "" H 9100 5350 50  0001 C CNN
+F 3 "" H 9100 5350 50  0001 C CNN
+	1    9100 5350
+	1    0    0    -1
+$EndComp
 $Comp
 L dp3t:SW_4PDT SW1
@@
 $EndComp
 Connection ~ 7800 5350
-Wire Wire Line
-	8500 5200 8500 5250
-Wire Wire Line
-	8500 5250 8700 5250
 $Comp
 L power:+BATT #PWR0110
@@
 $Comp
 L dp3t:SW_4PDT SW1
-U 1 1 5B19FE7B
+U 4 1 5B19FE7B
 P 7600 5350
 F 0 "SW1" H 7750 5650 50  0000 C CNN
@@
 F 2 "wemos:4PDT" H 7600 5350 50  0001 C CNN
 F 3 "" H 7600 5350 50  0001 C CNN
-	1    7600 5350
+	4    7600 5350
 	-1   0    0    -1
 $EndComp
@@
 	5400 7500 5750 7500
 Connection ~ 5750 7500
+Wire Wire Line
+	9100 5650 9100 5750
+Connection ~ 9100 5750
+Wire Wire Line
+	9100 5850 9100 6750
+$Comp
+L Connector_Generic:Conn_01x02 J3
+U 1 1 5B230E0E
+P 4200 4650
+F 0 "J3" H 4120 4867 50  0000 C CNN
+F 1 "Charge" H 4120 4776 50  0000 C CNN
+F 2 "Pin_Headers:Pin_Header_Angled_1x02_Pitch2.54mm" H 4200 4650 50  0001 C CNN
+F 3 "~" H 4200 4650 50  0001 C CNN
+	1    4200 4650
+	-1   0    0    -1
+$EndComp
+$Comp
+L power:+BATT #PWR0104
+U 1 1 5B230E14
+P 4400 4350
+F 0 "#PWR0104" H 4400 4200 50  0001 C CNN
+F 1 "+BATT" H 4415 4523 50  0000 C CNN
+F 2 "" H 4400 4350 50  0001 C CNN
+F 3 "" H 4400 4350 50  0001 C CNN
+	1    4400 4350
+	1    0    0    -1
+$EndComp
+$Comp
+L power:GND #PWR0112
+U 1 1 5B230E1A
+P 4400 4750
+F 0 "#PWR0112" H 4400 4500 50  0001 C CNN
+F 1 "GND" H 4405 4577 50  0000 C CNN
+F 2 "" H 4400 4750 50  0001 C CNN
+F 3 "" H 4400 4750 50  0001 C CNN
+	1    4400 4750
+	1    0    0    -1
+$EndComp
+Wire Wire Line
+	4400 4650 4400 4350
 $EndSCHEMATC
